Commit message: lidar and world test

File: description/robot.urdf.xacro (robot description, xacro)
@@ -1,6 +1,6 @@
 <?xml version="1.0"?>
 <robot xmlns:xacro="http://www.ros.org/wiki/xacro"  name="robot">
-    <xacro:include filename="inertial_macros.xacro" />
-    <!-- Example link -->
-    <xacro:include filename="robot_core.urdf.xacro" />
+    <xacro:include filename="robot_core.xacro" />
+    <xacro:include filename="gazebo_control.xacro" />
+    <xacro:include filename="lidar.xacro" />
 </robot>

File: description/robot_core.urdf.xacro (robot description, xacro)
@@ -50,5 +50,5 @@
         <parent link="base_link"/>
         <child link="left_wheel"/>
-        <origin xyz="0.0 0.175 0" rpy="-${pi/2} 0.0 0.0"/>
+        <origin xyz="0.0 0.175 0" rpy="0.0 0.0 ${-pi/2}"/>
         <axis xyz="0 0 1"/>
     </joint>
@@ -124,3 +124,49 @@
         </xacro:inertial_sphere>
     </link>
+    <!-- Add the depth camera -->
+    <joint name="camera_joint" type="fixed">
+        <parent link="base_link"/>
+        <child link="camera_link"/>
+        <origin xyz="0.25 0 0.2" rpy="0 0 0"/>
+    </joint>
+    <link name="camera_link">
+        <visual>
+            <origin xyz="0 0 0" rpy="0 0 0"/>
+            <geometry>
+                <box size="0.05 0.05 0.1"/>
+            </geometry>
+            <material name="black"/>
+        </visual>
+        <collision>
+            <origin xyz="0 0 0" rpy="0 0 0"/>
+            <geometry>
+                <box size="0.05 0.05 0.1"/>
+            </geometry>
+        </collision>
+    </link>
+    <!-- Gazebo simulation plugins -->
+    <gazebo>
+      <plugin name="gazebo_ros_control" filename="libgazebo_ros_control.so">
+        <robotNamespace>/</robotNamespace>
+      </plugin>
+    </gazebo>
+    <gazebo reference="base_link">
+      <static>true</static>
+    </gazebo>
+    <gazebo reference="left_wheel">
+      <mu1>10</mu1>
+      <mu2>10</mu2>
+      <kp>1000000.0</kp>
+      <kd>1.0</kd>
+      <minDepth>0.001</minDepth>
+      <maxVel>0.01</maxVel>
+    </gazebo>
+    <gazebo reference="right_wheel">
+      <mu1>10</mu1>
+      <mu2>10</mu2>
+      <kp>1000000.0</kp>
+      <kd>1.0</kd>
+      <minDepth>0.001</maxDepth>
+      <maxVel>0.01</maxVel>
+    </gazebo>
 </robot>
